Commit message: 已经可以训练平衡车，速度跟踪

File: genesis/assets/urdf/balance/urdf/wheelchair_description.urdf (robot description, URDF)
Before this commit: robot wheelchair_description, 3 links, 2 joints
Links:
- link base_link: geometry collision mesh filename=../meshes/base_link.STL; visual mesh filename=../meshes/base_link.STL
- link left_wheel: geometry collision mesh filename=../meshes/left_wheel.STL; visual mesh filename=../meshes/left_wheel.STL
- link right_wheel: geometry collision mesh filename=../meshes/right_wheel.STL; visual mesh filename=../meshes/right_wheel.STL
